File: main_board.sch (KiCad schematic (older format))
At the start: 5 parts, among them J101 Conn_Coaxial_x2, J102 Conn_Coaxial_x2, P101 PJRAS4X2U01AUX, P102 CONN_01X03, P103 HP_OUT_CONN_01X03

Commit message: Finished layout
Parts:
- removed P102: CONN_01X03, Pin_Headers_Female:Pin_Header_Straight_Female_1x03_Pitch2.54mm, symbol CONN_01X03
- removed P103: HP_OUT_CONN_01X03, Pin_Headers_Female:Pin_Header_Straight_Female_1x03_Pitch2.54mm, symbol CONN_01X03
- added J103, J104, J105: Conn_01x03_Male, Connectors_Molex:Molex_KK-6410-03_03x2.54mm_Straight, symbol Conn_01x03_Male
- P101: Mfg_part_# (none) -> PJRAS4X2U01AUX
Connections:
- net ASYM_OUT_L: now also J105.2 (Pin_2)
- net ASYM_OUT_R: now also J105.3 (Pin_3)
- net GND: now also P101.SA (GND), P101.SB (GND), P101.SC (GND), P101.SD (GND), J103.2 (Pin_2), J104.3 (Pin_3), J105.1 (Pin_1); no longer P101.SA (GND), P101.SB (GND), P101.SC (GND), P101.SD (GND)
- net V+: now also J103.1 (Pin_1)
- net V-: now also J103.3 (Pin_3)
- net headphone_preamp/OUT_L: now also J104.1 (Pin_1)
- net headphone_preamp/OUT_R: now also J104.2 (Pin_2)
- net preamp_1/Left_input: now also P101.T2D (L); no longer P101.T2A (L)
- net preamp_1/Right_input: now also P101.T1D (R); no longer P101.T1A (R)
- net preamp_2/Left_input: now also P101.T2C (L); no longer P101.T1B (R)
- net preamp_2/Right_input: now also P101.T1C (R); no longer P101.T2B (L)
- net preamp_3/Left_input: now also P101.T2B (L); no longer P101.T2C (L)
- net preamp_3/Right_input: now also P101.T1B (R); no longer P101.T1C (R)
- net preamp_4/Left_input: now also P101.T2A (L); no longer P101.T2D (L)
- net preamp_4/Right_input: now also P101.T1A (R); no longer P101.T1D (R)
Other:
- note added: "Power input\nMale Molex locking header\nshould be connected to a panel-mount DIN connector"
