File: master.sch (KiCad schematic (older format))
At the start: 18 parts, among them U701 NE5532

Commit message: Finished layout
Parts:
- added J701: Conn_01x05_Male, Connectors_Molex:Molex_KK-6410-05_05x2.54mm_Straight, symbol Conn_01x05_Male
- added J702: Conn_01x05_Female, symbol Conn_01x05_Female
- C701, C702: footprint (none) -> Capacitors_ThroughHole:C_Rect_L7.2mm_W3.5mm_P5.00mm_FKS2_FKP2_MKS2_MKP2; Description (none) -> Film Capacitors 400volts 0.010uF 5%; Distributor (none) -> Mouser; Distributor Part # (none) -> 80-R82MC2100Z350J; Manufacturer (none) -> Kemet; Mfg_Part_No (none) -> R82MC2100Z350J; Package (none) -> 0402
- C703, C704: footprint (none) -> w_capacitors:CP_5x11mm; Description (none) -> Aluminium Electrolytic Capacitors - Leaded 35volts 47uF 20%; Distributor (none) -> Mouser; Distributor Part # (none) -> 80-ESK476M035AC3EA; Manufacturer (none) -> Kemet; Mfg_Part_No (none) -> ESK476M035AC3EA; Package (none) -> 2-THT
- C705, C706: footprint (none) -> w_capacitors:CP_5x11mm; Description (none) -> Aluminium Electrolytic Capacitors - Leaded 16volts 22uF 20%; Distributor Part # (none) -> 80-ESE226M016AC3FA; Manufacturer (none) -> Kemet; Mfg_Part_No 0 -> ESE226M016AC3FA; Mfg_part_# (none) -> ESE226M016AC3FA; Package 0402 -> 2-THT
- C707, C708: footprint (none) -> w_capacitors:CP_5x11mm; Description (none) -> Aluminium Electrolytic Capacitors - Leaded 100volts 4.7uF 2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; Distributor (none) -> Mouser; Distributor Part # (none) -> 80-ESK475M100AC3FA; Manufacturer (none) -> Kemet; Mfg_Part_No (none) -> ESK475M100AC3FA; Mfg_part_# (none) -> ESK475M100AC3FA; Package (none) -> 2-THT
- R701, R702: footprint (none) -> Resistors_ThroughHole:R_Axial_DIN0204_L3.6mm_D1.6mm_P7.62mm_Horizontal; Distributor (none) -> Digikey; Mfg_Part_No (none) -> 0; Package (none) -> 0402
- R703, R704: Description (none) -> Résistances à couche métallique - Trou traversant 1/4watt 1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; Distributor Digikey -> Mouser; Distributor Part # (none) -> 71-CMF5010K000FKEB; Manufacturer (none) -> Vishay / Dale; Mfg_Part_No 0 -> CMF5010K000FKEB; Mfg_part_# (none) -> CMF5010K000FKEB
- R705, R706: Description (none) -> Résistances à couche métallique - Trou traversant 1/4watt 1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; Distributor Digikey -> Mouser; Distributor Part # (none) -> 71-CMF5012K100FHEB; Manufacturer (none) -> Vishay / Dale; Mfg_Part_No 0 -> CMF5012K100FHEB; Mfg_part_# (none) -> CMF5012K100FHEB; Package 0402 -> (none)
- R707, R708: footprint (none) -> Resistors_ThroughHole:R_Axial_DIN0204_L3.6mm_D1.6mm_P5.08mm_Horizontal; Distributor (none) -> Digikey; Mfg_Part_No (none) -> 0; Package (none) -> 0402
Connections:
- net GND: now also J701.3 (Pin_3), J702.3 (Pin_3)
- net V+: no longer C701.2, C703.1, R701.1, U701.8 (V+), U701.8 (V+)
- net V-: no longer C702.2, C704.2, R702.1, U701.4 (V-), U701.4 (V-)
- net PRE_MIX_R: now reaches R705.1, RV701.1, U701.1
- net PRE_MIX_R: now also J701.5 (Pin_5), J702.5 (Pin_5)
- net at C707.1: now also J701.2 (Pin_2); no longer RV701.2
- net PRE_MIX_L: now reaches R706.1, RV701.4, U701.7
- net PRE_MIX_L: now also J701.4 (Pin_4), J702.4 (Pin_4)
- net MIX_OUT_L: now reaches C708.1, RV701.5
- net MIX_OUT_L: now also J701.1 (Pin_1), J702.1 (Pin_1)
- new net +15V: C701.2, C703.1, R701.1, U701.8 (V+), U701.8 (V+)
- new net -15V: C702.2, C704.2, R702.1, U701.4 (V-), U701.4 (V-)
- new net MIX_OUT_R: J702.2 (Pin_2), RV701.2
Other:
- moved on the sheet: C707, R707, R708, RV701
