File: symetriseur.sch (KiCad schematic (older format))
At the start: 9 parts, among them J1201 Conn_01x03_Male, J1202 Conn_01x03_Male, J1203 XLR3, J1204 Conn_01x03_Female, J1205 XLR3, J1206 Conn_01x03_Female, SW1201 SW_DPST, T1201 Transformer_SP_2S, T1202 Transformer_SP_2S

Commit message: Finished layout
Parts:
- removed J1201, J1202: Conn_01x03_Male, Connectors_Molex:Molex_KK-6410-03_03x2.54mm_Straight, symbol Conn_01x03_Male
- removed J1204, J1206: Conn_01x03_Female, symbol Conn_01x03_Female
- added J1201: Conn_01x04_Male, Connectors_Molex:Molex_KK-6410-04_04x2.54mm_Straight, symbol Conn_01x04_Male
- added J1202: Conn_01x04_Female, symbol Conn_01x04_Female
- J1203, J1205: footprint (none) -> Neutrik:Neutrik_NC3MAAH-0; Description XLR Connectors 3P MALE VERT CHASS PANEL ISOL -> Connecteurs XLR 3P MALE HORIZ CHASS PANEL ISOL; Distributor Part # 568-NC3MAAV-0 -> 568-NC3MAAH-0; Mfg_Part_No NC3MAAV-0 -> NC3MAAH-0; Mfg_part_# (none) -> NC3MAAV-0
- SW1201: Mfg_part_# (none) -> SS-22F02-DG 6 (L)
- T1201, T1202: Mfg_part_# (none) -> TY-250P
Connections:
- net GND: now also J1201.1 (Pin_1), J1201.2 (Pin_2); no longer SW1201.1, SW1201.3
- net at J1203.2: now also T1201.7 (OUT2B)
- net at J1203.3: now also T1201.4 (OUT1A)
- net at J1205.2: now also T1202.7 (OUT2B)
- net at J1205.3: now also T1202.4 (OUT1A)
- net at SW1201.4: now also J1202.4 (Pin_4)
- net at SW1201.2: now also J1202.3 (Pin_3)
- net XLR_GND renamed XLR_GND_L
- net XLR_GND_L: now also J1201.4 (Pin_4); no longer J1203.1
- new net: J1202.2 (Pin_2), SW1201.1
- new net: J1202.1 (Pin_1), SW1201.3
- new net XLR_GND_R: J1201.3 (Pin_3), J1203.1
Other:
- moved on the sheet: J1203, SW1201
