File: main_board.kicad_pcb (KiCad board)
At the start: 2 copper layers, 280 x 180 mm, 25 parts, among them J101 Conn_Coaxial_x2, J102 Conn_Coaxial_x2, J1201 Conn_01x03_Male, J1202 Conn_01x03_Male, J1203 XLR3, J1205 XLR3, M301 Mixer, P101 PJRAS4X2U01AUX, P102 CONN_01X03, P103 HP_OUT_CONN_01X03, T1201 Transformer_SP_2S, T1202 Transformer_SP_2S, U701 NE5532

Commit message: Finished layout
Parts:
- removed H701, H702, H703: Header_01x03, Pin_Headers_Female:Pin_Header_Straight_Female_1x03_Pitch2.54mm
- removed J1202: Conn_01x03_Male, Connectors_Molex:Molex_KK-6410-03_03x2.54mm_Straight
- removed P102: CONN_01X03, Pin_Headers_Female:Pin_Header_Straight_Female_1x03_Pitch2.54mm
- removed P103 (x2): HP_OUT_CONN_01X03, Pin_Headers_Female:Pin_Header_Straight_Female_1x03_Pitch2.54mm
- added C701: 100n, Capacitors_ThroughHole:C_Rect_L7.2mm_W3.5mm_P5.00mm_FKS2_FKP2_MKS2_MKP2, F.Cu at (266.5, 194.2)
- added C702: 100n, Capacitors_ThroughHole:C_Rect_L7.2mm_W3.5mm_P5.00mm_FKS2_FKP2_MKS2_MKP2, F.Cu at (280.6, 193.8)
- added C703: 47u, w_capacitors:CP_5x11mm, F.Cu at (272.4, 192.7)
- added C704: 47u, w_capacitors:CP_5x11mm, F.Cu at (286.3, 192.3)
- added C705: 22u, w_capacitors:CP_5x11mm, F.Cu at (289.0, 165.6)
- added C706: 22u, w_capacitors:CP_5x11mm, F.Cu at (265.5, 163.2)
- added C707: 4u7, w_capacitors:CP_5x11mm, F.Cu at (275.3, 156.2)
- added C708: 4u7, w_capacitors:CP_5x11mm, F.Cu at (283.9, 156.2)
- added J103: Conn_01x03_Male, Connectors_Molex:Molex_KK-6410-03_03x2.54mm_Straight, F.Cu at (313.7, 60.0)
- added J104: Conn_01x03_Male, Connectors_Molex:Molex_KK-6410-03_03x2.54mm_Straight, F.Cu at (281.9, 218.0)
- added J105: Conn_01x03_Male, Connectors_Molex:Molex_KK-6410-03_03x2.54mm_Straight, F.Cu at (164.4, 61.5)
- added J1301: Conn_01x05_Male, Connectors_Molex:Molex_KK-6410-05_05x2.54mm_Straight, F.Cu at (90.0, 218.0)
- added J1401: Conn_01x05_Male, Connectors_Molex:Molex_KK-6410-05_05x2.54mm_Straight, F.Cu at (138.0, 218.0)
- added J1501: Conn_01x05_Male, Connectors_Molex:Molex_KK-6410-05_05x2.54mm_Straight, F.Cu at (188.0, 218.0)
- added J1601: Conn_01x05_Male, Connectors_Molex:Molex_KK-6410-05_05x2.54mm_Straight, F.Cu at (238.0, 218.0)
- added J701: Conn_01x05_Male, Connectors_Molex:Molex_KK-6410-05_05x2.54mm_Straight, F.Cu at (320.2, 145.1)
- added R1301: 100K, Resistors_ThroughHole:R_Axial_DIN0204_L3.6mm_D1.6mm_P5.08mm_Horizontal, F.Cu at (86.0, 204.9)
- added R1302: 100K, Resistors_ThroughHole:R_Axial_DIN0204_L3.6mm_D1.6mm_P5.08mm_Horizontal, F.Cu at (90.0, 204.9)
- added R1401: 100K, Resistors_ThroughHole:R_Axial_DIN0204_L3.6mm_D1.6mm_P5.08mm_Horizontal, F.Cu at (134.0, 204.9)
- added R1402: 100K, Resistors_ThroughHole:R_Axial_DIN0204_L3.6mm_D1.6mm_P5.08mm_Horizontal, F.Cu at (137.9, 204.9)
- added R1501: 100K, Resistors_ThroughHole:R_Axial_DIN0204_L3.6mm_D1.6mm_P5.08mm_Horizontal, F.Cu at (184.0, 204.9)
- added R1502: 100K, Resistors_ThroughHole:R_Axial_DIN0204_L3.6mm_D1.6mm_P5.08mm_Horizontal, F.Cu at (188.0, 204.9)
- added R1601: 100K, Resistors_ThroughHole:R_Axial_DIN0204_L3.6mm_D1.6mm_P5.08mm_Horizontal, F.Cu at (234.0, 204.9)
- added R1602: 100K, Resistors_ThroughHole:R_Axial_DIN0204_L3.6mm_D1.6mm_P5.08mm_Horizontal, F.Cu at (238.0, 204.9)
- added R701: 100, Resistors_ThroughHole:R_Axial_DIN0204_L3.6mm_D1.6mm_P7.62mm_Horizontal, F.Cu at (265.7, 185.8)
- added R702: 100, Resistors_ThroughHole:R_Axial_DIN0204_L3.6mm_D1.6mm_P7.62mm_Horizontal, F.Cu at (279.8, 185.7)
- added R703: 10K, Resistors_ThroughHole:R_Axial_DIN0204_L3.6mm_D1.6mm_P5.08mm_Horizontal, F.Cu at (284.9, 171.0)
- added R704: 10K, Resistors_ThroughHole:R_Axial_DIN0204_L3.6mm_D1.6mm_P5.08mm_Horizontal, F.Cu at (269.5, 168.3)
- added R705: 12K, Resistors_ThroughHole:R_Axial_DIN0204_L3.6mm_D1.6mm_P5.08mm_Horizontal, F.Cu at (284.9, 173.8)
- added R706: 12K, Resistors_ThroughHole:R_Axial_DIN0204_L3.6mm_D1.6mm_P5.08mm_Horizontal, F.Cu at (269.5, 171.0)
- added R707: R_Small, Resistors_ThroughHole:R_Axial_DIN0204_L3.6mm_D1.6mm_P5.08mm_Horizontal, F.Cu at (276.4, 144.2)
- added R708: R_Small, Resistors_ThroughHole:R_Axial_DIN0204_L3.6mm_D1.6mm_P5.08mm_Horizontal, F.Cu at (283.1, 144.3)
- added REF**: MountingHole_4.3mm_M4, Mounting_Holes:MountingHole_4.3mm_M4, F.Cu at (57.0, 57.0)
- added REF**: MountingHole_4.3mm_M4, Mounting_Holes:MountingHole_4.3mm_M4, F.Cu at (57.0, 223.0)
- added REF**: MountingHole_4.3mm_M4, Mounting_Holes:MountingHole_4.3mm_M4, F.Cu at (323.0, 223.0)
- added REF**: MountingHole_4.3mm_M4, Mounting_Holes:MountingHole_4.3mm_M4, F.Cu at (323.0, 57.0)
- J1201: value Conn_01x03_Male -> Conn_01x04_Male; footprint Connectors_Molex:Molex_KK-6410-03_03x2.54mm_Straight -> Connectors_Molex:Molex_KK-6410-04_04x2.54mm_Straight
- J1203, J1205: footprint Neutrik:Neutrik_NC3MAAH-1 -> Neutrik:Neutrik_NC3MAAH-0
- moved U701 22.5 mm to (280.9, 173.5), turned to 180 degrees
- moved J1201 15.3 mm to (223.8, 64.0), turned to 90 degrees
- moved M301 12.4 mm to (158.0, 181.8)
- moved A801 9.28 mm to (299.2, 176.9)
- moved C401 8.88 mm to (158.0, 161.9)
- moved B501 7.96 mm to (158.0, 142.4)
- moved J1205 6.60 mm to (273.0, 50.0)
- moved R201 6.46 mm to (90.0, 75.0)
- moved R1101 4.87 mm to (291.0, 75.0)
- moved R901 3.72 mm to (157.0, 75.0)
- moved ISO601 3.70 mm to (158.0, 124.9)
- moved R1001 3.05 mm to (224.0, 75.0)
- moved J1203 2.45 mm to (243.4, 50.0)
- moved T1202 2.23 mm to (312.0, 129.0)
- moved T1201 1.86 mm to (279.0, 129.0)
Connections:
- B501 pad 11: /PO2_L -> /TO2_L
- B501 pad 12: /PO2_R -> /TO2_R
- B501 pad 18: /PO3_L -> /TO3_L
- B501 pad 19: /PO3_R -> /TO3_R
- B501 pad 25: /PO4_L -> /TO4_L
- B501 pad 26: /PO4_R -> /TO4_R
- B501 pad 4: /PO1_L -> /TO1_L
- B501 pad 5: /PO1_R -> /TO1_R
- J1201 pad 1: Net-(J1201-Pad1) -> GND
- J1201 pad 2: (no net) -> GND
- J1201 pad 3: Net-(J1201-Pad3) -> /symetriseur/XLR_GND_R
- J1203 pad 1: /symetriseur/XLR_GND -> /symetriseur/XLR_GND_R
- J1203 pad 2: (no net) -> Net-(J1203-Pad2)
- J1205 pad 1: /symetriseur/XLR_GND -> /symetriseur/XLR_GND_L
- J1205 pad 2: (no net) -> Net-(J1205-Pad2)
- P101 pad T1A: /preamp_1/Right_input -> /preamp_4/Right_input
- P101 pad T1B: /preamp_2/Left_input -> /preamp_3/Right_input
- P101 pad T1C: /preamp_3/Right_input -> /preamp_2/Right_input
- P101 pad T1D: /preamp_4/Right_input -> /preamp_1/Right_input
- P101 pad T2A: /preamp_1/Left_input -> /preamp_4/Left_input
- P101 pad T2B: /preamp_2/Right_input -> /preamp_3/Left_input
- P101 pad T2C: /preamp_3/Left_input -> /preamp_2/Left_input
- P101 pad T2D: /preamp_4/Left_input -> /preamp_1/Left_input
- T1201 pad 4: Net-(J1201-Pad3) -> Net-(J1203-Pad3)
- T1201 pad 7: Net-(J1201-Pad1) -> Net-(J1203-Pad2)
- T1202 pad 4: Net-(J1202-Pad3) -> Net-(J1205-Pad3)
- T1202 pad 7: Net-(J1202-Pad1) -> Net-(J1205-Pad2)
- U701 pad 1: (no net) -> /master/PRE_MIX_R
- U701 pad 2: (no net) -> Net-(R703-Pad1)
- U701 pad 4: /V- -> /master/-15V
- U701 pad 6: (no net) -> Net-(R704-Pad1)
- U701 pad 7: (no net) -> /master/PRE_MIX_L
- U701 pad 8: /V+ -> /master/+15V
Routing:
- net GND: track 0.00 -> 1577.0 mm, vias 0 -> 4
- net /V+: track 0.00 -> 758.1 mm, vias 0 -> 8
- net /V-: track 0.00 -> 718.6 mm, vias 0 -> 3
- net /MIX_OUT_L: track 0.00 -> 371.4 mm, vias 0 -> 1
- net /MIX_OUT_R: track 0.00 -> 367.1 mm, vias 0 -> 1
- net /CUE_OUT_L: track 0.00 -> 318.3 mm, vias 0 -> 1
- net /CUE_OUT_R: track 0.00 -> 304.5 mm, vias 0 -> 1
- net /ISO_OUT_R: track 0.00 -> 222.9 mm
- net /preamp_4/Right_input: track 0.00 -> 213.0 mm, vias 0 -> 1
- net /ISO_OUT_L: track 0.00 -> 200.2 mm
- net /ASYM_OUT_L: track 0.00 -> 192.3 mm, vias 0 -> 1
- net /PO4_R: track 0.00 -> 178.5 mm, vias 0 -> 1
- net /PO1_L: track 0.00 -> 159.7 mm, vias 0 -> 2
- net /preamp_4/Left_input: track 0.00 -> 159.5 mm, vias 0 -> 1
- net /preamp_3/Right_input: track 0.00 -> 159.2 mm, vias 0 -> 1
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- added copper zone on B.Cu, net GND
- added copper zone on F.Cu, net GND
Other:
- net class Default: trace_width 0.25 -> 0.7; via_dia 0.6 -> 0.7
- net class Masse: clearance 0.2 -> 0.25; trace_width 0.5 -> 1; via_dia 0.6 -> 1; via_drill 0.4 -> 0.6
- net class Power added: clearance 0.25, trace_width 1, via_dia 1, via_drill 0.6
- board text added: "-15V GND +15V"
- board text added: "CH1 RIAA"
- board text added: "CH2 RIAA"
- board text added: "CUE"
- board text added: "D&D"
- board text added: "EQ"
- board text added: "GND L R"
- board text added: "GND R L"
- board text added: "GND lift DPST"
- board text added: "HEADPHONE AMP"
- board text added: "HEADPHONE JACK CONN"
- board text added: "ISOLATOR"
- board text added: "MIXER"
- board text added: "Power IN"
- board text added: "RM4 main board 4818"
- board text added: "VU meter"
- board text added: "XLR L"
- board text added: "XLR R"

Commit message: Update silkscreen on RIAA footprints
Other:
- board text added: "CH3 RIAA"
- board text added: "CH4 RIAA"
Changed lines of the file:
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@@
 (kicad_pcb (version 4) (host pcbnew 4.0.7)
   (general
-    (links 0)
-    (no_connects 9)
-    (area 48.58 48.58 331.330001 231.330001)
+    (links 174)
+    (no_connects 3)
+    (area 47.392857 40.655 349.994286 231.330001)
     (thickness 1.6)
     (drawings 30)
@@
     (effects (font (size 1.5 1.5) (thickness 0.3)))
   )
-  (gr_text "CH1 RIAA\n" (at 291 91) (layer F.SilkS)
+  (gr_text "CH4 RIAA\n" (at 291 91) (layer F.SilkS)
     (effects (font (size 2 2) (thickness 0.3)))
   )
-  (gr_text "CH1 RIAA\n" (at 224 91) (layer F.SilkS)
+  (gr_text "CH3 RIAA\n" (at 224 91) (layer F.SilkS)
     (effects (font (size 2 2) (thickness 0.3)))
   )
